File: battery-protector-v2.sch (KiCad schematic (older format))
At the start: 25 parts, among them J1 Conn_01x04, J2 Anderson_two_redblack, J3 Anderson_two_redblack, P1 USB_B_POWER_SUPPLY, SW1 SW_SPST, SW2 SW_SPDT, U1 SAMD21E18, U2 WS2812b, U3 MIC5203, U4 MOSFET_N

Commit message: Added footprints
Parts:
- removed R8: 10, symbol R
- removed U4: MOSFET_N, symbol MOSFET_N
- added H1, H2, H3, H4: HOLE, homebrew:HOLE_M4, symbol HOLE
- added U4: MOSFET_CSD17318Q2, homebrew:TRANS_CSD17318Q2T, symbol MOSFET_CSD17318Q2
- D1: value D -> BAT54GWJ; footprint (none) -> Diodes_SMD:D_SOD-123
- D2: value D -> S10KCV7G; footprint (none) -> homebrew:DIODE-DO-214AB
- F1: value POWER_FUSE -> BK-6010; footprint FUSE_5MM -> homebrew:FUSEHOLDER_ATC_Bk-6010
- J2, J3: footprint (none) -> homebrew:Anderson_1337G3_right_angle_bottom_two
- P1: value USB_B_POWER_SUPPLY -> 10118194; footprint (none) -> 10118194-0001LF:FRAMATOME_10118194-0001LF
- R1: value 220 -> 470; footprint (none) -> Resistors_SMD:R_0603
- R2, R3, R5, R6, R7: footprint (none) -> Resistors_SMD:R_0603
- R4: footprint (none) -> homebrew:R_PHOTO
- RV1: footprint (none) -> homebrew:BOURNS_PDB12H_POT
- SW1: footprint (none) -> Sparkfun-Switches:TACTILE_SWITCH_SMD_4.6X2.8MM
- SW2: value SW_SPDT -> OS102011MS2QN1; footprint (none) -> homebrew:SW_2POS_OS102011MS2QN1
- U2: footprint (none) -> homebrew:WS2812B
Changed lines of the file:
@@
 F 0 "SW1" H 900 1475 50  0000 C CNN
 F 1 "SW_SPST" H 900 1250 50  0000 C CNN
-F 2 "" H 900 1350 50  0001 C CNN
+F 2 "Sparkfun-Switches:TACTILE_SWITCH_SMD_4.6X2.8MM" H 900 1350 50  0001 C CNN
 F 3 "" H 900 1350 50  0001 C CNN
 	1    900  1350
@@
 P 1450 7150
 F 0 "P1" H 1650 6950 50  0000 C CNN
-F 1 "USB_B_POWER_SUPPLY" H 1400 7350 50  0000 C CNN
-F 2 "" V 1400 7050 50  0001 C CNN
+F 1 "10118194" H 1400 7350 50  0000 C CNN
+F 2 "10118194-0001LF:FRAMATOME_10118194-0001LF" V 1400 7050 50  0001 C CNN
 F 3 "" V 1400 7050 50  0000 C CNN
 	1    1450 7150
@@
 F 0 "J2" H 10150 750 60  0000 C CNN
 F 1 "Anderson_two_redblack" H 10150 1050 60  0000 C CNN
-F 2 "" H 10100 750 60  0001 C CNN
+F 2 "homebrew:Anderson_1337G3_right_angle_bottom_two" H 10100 750 60  0001 C CNN
 F 3 "" H 10100 750 60  0001 C CNN
 	1    10150 900
@@
 F 0 "J3" H 10150 1350 60  0000 C CNN
 F 1 "Anderson_two_redblack" H 10150 1650 60  0000 C CNN
-F 2 "" H 10100 1350 60  0001 C CNN
+F 2 "homebrew:Anderson_1337G3_right_angle_bottom_two" H 10100 1350 60  0001 C CNN
 F 3 "" H 10100 1350 60  0001 C CNN
 	1    10150 1500
@@
 P 9100 850
 F 0 "F1" H 8700 950 50  0000 L BNN
-F 1 "POWER_FUSE" H 9300 950 50  0000 L BNN
-F 2 "FUSE_5MM" H 9130 1000 20  0001 C CNN
+F 1 "BK-6010" H 9300 950 50  0000 L BNN
+F 2 "homebrew:FUSEHOLDER_ATC_Bk-6010" H 9130 1000 20  0001 C CNN
 F 3 "" H 9100 850 60  0000 C CNN
 	1    9100 850
@@
 F 0 "R4" H 5350 1600 50  0000 L CNN
 F 1 "R_PHOTO" H 5350 1550 50  0000 L TNN
-F 2 "" V 5350 1300 50  0001 L CNN
+F 2 "homebrew:R_PHOTO" V 5350 1300 50  0001 L CNN
 F 3 "" H 5300 1500 50  0001 C CNN
 	1    5300 1550
@@
 F 0 "R5" V 5380 1950 50  0000 C CNN
 F 1 "16k" V 5300 1950 50  0000 C CNN
-F 2 "" V 5230 1950 50  0001 C CNN
+F 2 "Resistors_SMD:R_0603" V 5230 1950 50  0001 C CNN
 F 3 "" H 5300 1950 50  0001 C CNN
 	1    5300 1950
@@
 F 0 "R6" V 6030 1550 50  0000 C CNN
 F 1 "33k" V 5950 1550 50  0000 C CNN
-F 2 "" V 5880 1550 50  0001 C CNN
+F 2 "Resistors_SMD:R_0603" V 5880 1550 50  0001 C CNN
 F 3 "" H 5950 1550 50  0001 C CNN
 	1    5950 1550
@@
 F 0 "R7" V 6030 1950 50  0000 C CNN
 F 1 "10k" V 5950 1950 50  0000 C CNN
-F 2 "" V 5880 1950 50  0001 C CNN
+F 2 "Resistors_SMD:R_0603" V 5880 1950 50  0001 C CNN
 F 3 "" H 5950 1950 50  0001 C CNN
 	1    5950 1950
@@
 	1    0    0    -1
 $EndComp
-$Comp
-L MOSFET_N U4
-U 1 1 5B5145FE
-P 5400 3500
-F 0 "U4" H 5400 3600 60  0000 C CNN
-F 1 "MOSFET_N" H 5400 3500 60  0000 C CNN
-F 2 "" H 5400 3450 60  0000 C CNN
-F 3 "" H 5400 3450 60  0000 C CNN
-	1    5400 3500
-	0    -1   -1   0
-$EndComp
 Text GLabel 2250 1850 2    60   Input ~ 0
 VOUT_SIGNAL
@@
 F 0 "R2" V 4830 3650 50  0000 C CNN
 F 1 "10k" V 4750 3650 50  0000 C CNN
-F 2 "" V 4680 3650 50  0001 C CNN
+F 2 "Resistors_SMD:R_0603" V 4680 3650 50  0001 C CNN
 F 3 "" H 4750 3650 50  0001 C CNN
 	1    4750 3650
@@
 P 4600 3500
 F 0 "R1" V 4680 3500 50  0000 C CNN
-F 1 "220" V 4600 3500 50  0000 C CNN
-F 2 "" V 4530 3500 50  0001 C CNN
+F 1 "470" V 4600 3500 50  0000 C CNN
+F 2 "Resistors_SMD:R_0603" V 4530 3500 50  0001 C CNN
 F 3 "" H 4600 3500 50  0001 C CNN
 	1    4600 3500
@@
 P 5700 3150
 F 0 "D2" H 5700 3250 50  0000 C CNN
-F 1 "D" H 5700 3050 50  0000 C CNN
-F 2 "" H 5700 3150 50  0001 C CNN
+F 1 "S10KCV7G" H 5700 3050 50  0000 C CNN
+F 2 "homebrew:DIODE-DO-214AB" H 5700 3150 50  0001 C CNN
 F 3 "" H 5700 3150 50  0001 C CNN
 	1    5700 3150
@@
 L +BATT #PWR021
 U 1 1 5B515890
-P 6200 3100
-F 0 "#PWR021" H 6200 2950 50  0001 C CNN
-F 1 "+BATT" H 6200 3240 50  0000 C CNN
-F 2 "" H 6200 3100 50  0001 C CNN
-F 3 "" H 6200 3100 50  0001 C CNN
-	1    6200 3100
+P 5900 3100
+F 0 "#PWR021" H 5900 2950 50  0001 C CNN
+F 1 "+BATT" H 5900 3240 50  0000 C CNN
+F 2 "" H 5900 3100 50  0001 C CNN
+F 3 "" H 5900 3100 50  0001 C CNN
+	1    5900 3100
 	1    0    0    -1
 $EndComp
 Wire Wire Line
 	5550 3150 5300 3150
-$Comp
-L R R8
-U 1 1 5B515BEB
-P 6000 3150
-F 0 "R8" V 6080 3150 50  0000 C CNN
-F 1 "10" V 6000 3150 50  0000 C CNN
-F 2 "" V 5930 3150 50  0001 C CNN
-F 3 "" H 6000 3150 50  0001 C CNN
-	1    6000 3150
-	0    1    1    0
-$EndComp
-Wire Wire Line
-	6200 3100 6200 3150
-Wire Wire Line
-	6200 3150 6150 3150
+Wire Wire Line
+	5900 3100 5900 3150
+Wire Wire Line
+	5900 3150 5850 3150
 Text GLabel 2250 1750 2    60   Input ~ 0
 LED
@@
 F 0 "U2" H 2500 4600 60  0000 C CNN
 F 1 "WS2812b" H 2500 5150 60  0000 C CNN
-F 2 "" H 2500 4300 60  0001 C CNN
+F 2 "homebrew:WS2812B" H 2500 4300 60  0001 C CNN
 F 3 "" H 2500 4300 60  0001 C CNN
 	1    2550 4900
@@
 P 1100 6750
 F 0 "D1" H 1100 6850 50  0000 C CNN
-F 1 "D" H 1100 6650 50  0000 C CNN
-F 2 "" H 1100 6750 50  0001 C CNN
+F 1 "BAT54GWJ" H 1100 6650 50  0000 C CNN
+F 2 "Diodes_SMD:D_SOD-123" H 1100 6750 50  0001 C CNN
 F 3 "" H 1100 6750 50  0001 C CNN
 	1    1100 6750
@@
 P 5400 4850
 F 0 "SW2" H 5400 5020 50  0000 C CNN
-F 1 "SW_SPDT" H 5400 4650 50  0000 C CNN
-F 2 "" H 5400 4850 50  0001 C CNN
+F 1 "OS102011MS2QN1" H 5400 4650 50  0000 C CNN
+F 2 "homebrew:SW_2POS_OS102011MS2QN1" H 5400 4850 50  0001 C CNN
 F 3 "" H 5400 4850 50  0001 C CNN
 	1    5400 4850
@@
 F 0 "R3" V 5130 4850 50  0000 C CNN
 F 1 "10k" V 5050 4850 50  0000 C CNN
-F 2 "" V 4980 4850 50  0001 C CNN
+F 2 "Resistors_SMD:R_0603" V 4980 4850 50  0001 C CNN
 F 3 "" H 5050 4850 50  0001 C CNN
 	1    5050 4850
@@
 F 0 "RV1" V 6375 4850 50  0000 C CNN
 F 1 "POT" V 6450 4850 50  0000 C CNN
-F 2 "" H 6550 4850 50  0001 C CNN
+F 2 "homebrew:BOURNS_PDB12H_POT" H 6550 4850 50  0001 C CNN
 F 3 "" H 6550 4850 50  0001 C CNN
 	1    6550 4850
@@
 NoConn ~ 1550 7450
 NoConn ~ 2050 5050
+$Comp
+L MOSFET_CSD17318Q2 U4
+U 1 1 5B515988
+P 5400 3500
+F 0 "U4" H 5400 3600 60  0000 C CNN
+F 1 "MOSFET_CSD17318Q2" H 5400 3500 60  0000 C CNN
+F 2 "homebrew:TRANS_CSD17318Q2T" H 5400 3450 60  0001 C CNN
+F 3 "" H 5400 3450 60  0000 C CNN
+	1    5400 3500
+	0    -1   -1   0
+$EndComp
+$Comp
+L HOLE H1
+U 1 1 5B516C22
+P 9100 3900
+F 0 "H1" H 9100 3770 60  0000 C CNN
+F 1 "HOLE" H 9100 4020 60  0000 C CNN
+F 2 "homebrew:HOLE_M4" H 9100 3900 60  0001 C CNN
+F 3 "" H 9100 3900 60  0001 C CNN
+	1    9100 3900
+	1    0    0    -1
+$EndComp
+$Comp
+L HOLE H3
+U 1 1 5B516CA2
+P 9350 3900
+F 0 "H3" H 9350 3770 60  0000 C CNN
+F 1 "HOLE" H 9350 4020 60  0000 C CNN
+F 2 "homebrew:HOLE_M4" H 9350 3900 60  0001 C CNN
+F 3 "" H 9350 3900 60  0001 C CNN
+	1    9350 3900
+	1    0    0    -1
+$EndComp
+$Comp
+L HOLE H2
+U 1 1 5B516D0A
+P 9100 4250
+F 0 "H2" H 9100 4120 60  0000 C CNN
+F 1 "HOLE" H 9100 4370 60  0000 C CNN
+F 2 "homebrew:HOLE_M4" H 9100 4250 60  0001 C CNN
+F 3 "" H 9100 4250 60  0001 C CNN
+	1    9100 4250
+	1    0    0    -1
+$EndComp
+$Comp
+L HOLE H4
+U 1 1 5B516D75
+P 9350 4250
+F 0 "H4" H 9350 4120 60  0000 C CNN
+F 1 "HOLE" H 9350 4370 60  0000 C CNN
+F 2 "homebrew:HOLE_M4" H 9350 4250 60  0001 C CNN
+F 3 "" H 9350 4250 60  0001 C CNN
+	1    9350 4250
+	1    0    0    -1
+$EndComp
 $EndSCHEMATC
