File: hvac-v2.sch (KiCad schematic (older format))
At the start: 39 parts, among them J1 Conn_01x04, J2 Anderson_two_redblack, J3 Anderson_two_redblack, J4 Anderson_two_redblack, P1 10118194, P2 CONN_01X08, SW1 SW_SPST, SW2 SP3T, SW3 SW_PUSH, SW4 SW_PUSH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

Commit message: Switch to a potentiometer for mode control
Parts:
- removed R3, R4: 10k, Resistors_SMD:R_0603, symbol R
- removed SW2: SP3T, symbol SP3T
- added RV2: POT, homebrew:BOURNS_PDB12H_POT, symbol POT-RESCUE-hvac-v2
- P2: footprint (none) -> homebrew:1985250_phoenix_8pos_3.5mm
- U8: footprint TO-92-AMMO -> homebrew:TO-92
Connections:
- net GND: now also RV2.3
- net VCC: now also RV2.1
- net MODE_SW renamed MODE
- net MODE: now also RV2.2
Other:
- moved on the sheet: SW3, SW4
Changed lines of the file:
@@
 $EndComp
 Text GLabel 2250 1450 2    60   Input ~ 0
-MODE_SW
-$Comp
-L GND #PWR021
-U 1 1 5B517976
-P 4300 5400
-F 0 "#PWR021" H 4300 5150 50  0001 C CNN
-F 1 "GND" H 4300 5250 50  0000 C CNN
-F 2 "" H 4300 5400 50  0001 C CNN
-F 3 "" H 4300 5400 50  0001 C CNN
-	1    4300 5400
-	1    0    0    -1
-$EndComp
+MODE
 Text GLabel 2250 1550 2    60   Input ~ 0
 KNOB
@@
 $EndComp
 $Comp
-L VCC #PWR022
+L VCC #PWR021
 U 1 1 5B518324
 P 5350 5000
-F 0 "#PWR022" H 5350 4850 50  0001 C CNN
+F 0 "#PWR021" H 5350 4850 50  0001 C CNN
 F 1 "VCC" H 5350 5150 50  0000 C CNN
 F 2 "" H 5350 5000 50  0001 C CNN
@@
 $EndComp
 $Comp
-L GND #PWR023
+L GND #PWR022
 U 1 1 5B51837A
 P 5350 5300
-F 0 "#PWR023" H 5350 5050 50  0001 C CNN
+F 0 "#PWR022" H 5350 5050 50  0001 C CNN
 F 1 "GND" H 5350 5150 50  0000 C CNN
 F 2 "" H 5350 5300 50  0001 C CNN
@@
 $EndComp
 $Comp
-L VCC #PWR024
+L VCC #PWR023
 U 1 1 5B52A77C
 P 1550 5100
-F 0 "#PWR024" H 1550 4950 50  0001 C CNN
+F 0 "#PWR023" H 1550 4950 50  0001 C CNN
 F 1 "VCC" H 1550 5250 50  0000 C CNN
 F 2 "" H 1550 5100 50  0001 C CNN
@@
 $EndComp
 $Comp
-L GND #PWR025
+L GND #PWR024
 U 1 1 5B52A782
 P 2500 5350
-F 0 "#PWR025" H 2500 5100 50  0001 C CNN
+F 0 "#PWR024" H 2500 5100 50  0001 C CNN
 F 1 "GND" H 2500 5200 50  0000 C CNN
 F 2 "" H 2500 5350 50  0001 C CNN
@@
 $EndComp
 $Comp
-L VCC #PWR026
+L VCC #PWR025
 U 1 1 5B52A859
 P 1550 5750
-F 0 "#PWR026" H 1550 5600 50  0001 C CNN
+F 0 "#PWR025" H 1550 5600 50  0001 C CNN
 F 1 "VCC" H 1550 5900 50  0000 C CNN
 F 2 "" H 1550 5750 50  0001 C CNN
@@
 $EndComp
 $Comp
-L GND #PWR027
+L GND #PWR026
 U 1 1 5B52A85F
 P 2500 6000
-F 0 "#PWR027" H 2500 5750 50  0001 C CNN
+F 0 "#PWR026" H 2500 5750 50  0001 C CNN
 F 1 "GND" H 2500 5850 50  0000 C CNN
 F 2 "" H 2500 6000 50  0001 C CNN
@@
 PUMP_OUT
 $Comp
-L +BATT #PWR028
+L +BATT #PWR027
 U 1 1 5B515220
 P 9450 1450
-F 0 "#PWR028" H 9450 1300 50  0001 C CNN
+F 0 "#PWR027" H 9450 1300 50  0001 C CNN
 F 1 "+BATT" H 9450 1590 50  0000 C CNN
 F 2 "" H 9450 1450 50  0001 C CNN
@@
 $EndComp
 $Comp
-L +BATT #PWR029
+L +BATT #PWR028
 U 1 1 5B52B12B
 P 9450 1900
-F 0 "#PWR029" H 9450 1750 50  0001 C CNN
+F 0 "#PWR028" H 9450 1750 50  0001 C CNN
 F 1 "+BATT" H 9450 2040 50  0000 C CNN
 F 2 "" H 9450 1900 50  0001 C CNN
@@
 $EndComp
 $Comp
-L GND #PWR030
+L GND #PWR029
 U 1 1 5B52BE12
 P 4900 1800
-F 0 "#PWR030" H 4900 1550 50  0001 C CNN
+F 0 "#PWR029" H 4900 1550 50  0001 C CNN
 F 1 "GND" H 4900 1650 50  0000 C CNN
 F 2 "" H 4900 1800 50  0001 C CNN
@@
 $EndComp
 $Comp
-L GND #PWR031
+L GND #PWR030
 U 1 1 5B52BE1E
 P 5450 1950
-F 0 "#PWR031" H 5450 1700 50  0001 C CNN
+F 0 "#PWR030" H 5450 1700 50  0001 C CNN
 F 1 "GND" H 5450 1800 50  0000 C CNN
 F 2 "" H 5450 1950 50  0001 C CNN
@@
 $EndComp
 $Comp
-L +BATT #PWR032
+L +BATT #PWR031
 U 1 1 5B52BE2F
 P 6050 1100
-F 0 "#PWR032" H 6050 950 50  0001 C CNN
+F 0 "#PWR031" H 6050 950 50  0001 C CNN
 F 1 "+BATT" H 6050 1240 50  0000 C CNN
 F 2 "" H 6050 1100 50  0001 C CNN
@@
 L SW_PUSH SW3
 U 1 1 5B52C4F4
-P 6450 5050
-F 0 "SW3" H 6600 5160 50  0000 C CNN
-F 1 "SW_PUSH" H 6450 4970 50  0000 C CNN
-F 2 "" H 6450 5050 50  0000 C CNN
-F 3 "" H 6450 5050 50  0000 C CNN
-	1    6450 5050
+P 7000 5050
+F 0 "SW3" H 7150 5160 50  0000 C CNN
+F 1 "SW_PUSH" H 7000 4970 50  0000 C CNN
+F 2 "" H 7000 5050 50  0001 C CNN
+F 3 "" H 7000 5050 50  0000 C CNN
+	1    7000 5050
 	1    0    0    -1
 $EndComp
@@
 F 0 "SW5" H 9000 950 50  0000 C CNN
 F 1 "SPST" H 9000 750 50  0000 C CNN
-F 2 "" H 9000 850 50  0000 C CNN
+F 2 "" H 9000 850 50  0001 C CNN
 F 3 "" H 9000 850 50  0000 C CNN
 	1    9000 850
@@
 $EndComp
 $Comp
-L GND #PWR033
+L GND #PWR032
 U 1 1 5B52D407
-P 6150 5050
-F 0 "#PWR033" H 6150 4800 50  0001 C CNN
-F 1 "GND" H 6150 4900 50  0000 C CNN
-F 2 "" H 6150 5050 50  0000 C CNN
-F 3 "" H 6150 5050 50  0000 C CNN
-	1    6150 5050
-	1    0    0    -1
-$EndComp
-Text GLabel 6750 5050 2    60   Input ~ 0
+P 6700 5050
+F 0 "#PWR032" H 6700 4800 50  0001 C CNN
+F 1 "GND" H 6700 4900 50  0000 C CNN
+F 2 "" H 6700 5050 50  0000 C CNN
+F 3 "" H 6700 5050 50  0000 C CNN
+	1    6700 5050
+	1    0    0    -1
+$EndComp
+Text GLabel 7300 5050 2    60   Input ~ 0
 NAP_BUTTON
 Text GLabel 2250 2150 2    60   Input ~ 0
 NAP_BUTTON
-$Comp
-L SP3T SW2
-U 1 1 5B52E3A7
-P 4000 5150
-F 0 "SW2" H 3900 5300 50  0000 C CNN
-F 1 "SP3T" H 3900 5050 50  0000 C CNN
-F 2 "" H 3375 5325 50  0000 C CNN
-F 3 "" H 3375 5325 50  0000 C CNN
-	1    4000 5150
-	1    0    0    -1
-$EndComp
-Text GLabel 3700 5150 0    60   Input ~ 0
-MODE_SW
-$Comp
-L R R3
-U 1 1 5B5177BF
-P 4400 5000
-F 0 "R3" V 4480 5000 50  0000 C CNN
-F 1 "10k" V 4400 5000 50  0000 C CNN
-F 2 "Resistors_SMD:R_0603" V 4330 5000 50  0001 C CNN
-F 3 "" H 4400 5000 50  0001 C CNN
-	1    4400 5000
-	1    0    0    -1
-$EndComp
-$Comp
-L R R4
-U 1 1 5B52F3C3
-P 4700 5100
-F 0 "R4" V 4780 5100 50  0000 C CNN
-F 1 "10k" V 4700 5100 50  0000 C CNN
-F 2 "Resistors_SMD:R_0603" V 4630 5100 50  0001 C CNN
-F 3 "" H 4700 5100 50  0001 C CNN
-	1    4700 5100
-	-1   0    0    1
-$EndComp
-$Comp
-L VCC #PWR034
-U 1 1 5B517923
-P 4300 4850
-F 0 "#PWR034" H 4300 4700 50  0001 C CNN
-F 1 "VCC" H 4300 5000 50  0000 C CNN
-F 2 "" H 4300 4850 50  0001 C CNN
-F 3 "" H 4300 4850 50  0001 C CNN
-	1    4300 4850
-	1    0    0    -1
-$EndComp
+Text GLabel 4200 5150 2    60   Input ~ 0
+MODE
 Wire Wire Line
 	1100 1050 1150 1050
@@
 Wire Wire Line
 	6050 1150 6000 1150
-Wire Wire Line
-	4300 4850 4300 5050
-Wire Wire Line
-	4300 4850 4400 4850
-Wire Wire Line
-	4300 5150 4550 5150
-Wire Wire Line
-	4550 5150 4550 4950
-Wire Wire Line
-	4550 4950 4700 4950
-Wire Wire Line
-	4700 5250 4300 5250
-Connection ~ 4400 5150
-Wire Wire Line
-	4300 5250 4300 5400
 $Comp
 L SW_PUSH SW4
 U 1 1 5B531467
-P 6450 5350
-F 0 "SW4" H 6600 5460 50  0000 C CNN
-F 1 "SW_PUSH" H 6450 5270 50  0000 C CNN
-F 2 "" H 6450 5350 50  0000 C CNN
-F 3 "" H 6450 5350 50  0000 C CNN
-	1    6450 5350
-	1    0    0    -1
-$EndComp
-$Comp
-L GND #PWR035
+P 7000 5350
+F 0 "SW4" H 7150 5460 50  0000 C CNN
+F 1 "SW_PUSH" H 7000 5270 50  0000 C CNN
+F 2 "" H 7000 5350 50  0001 C CNN
+F 3 "" H 7000 5350 50  0000 C CNN
+	1    7000 5350
+	1    0    0    -1
+$EndComp
+$Comp
+L GND #PWR033
 U 1 1 5B53146D
-P 6150 5350
-F 0 "#PWR035" H 6150 5100 50  0001 C CNN
-F 1 "GND" H 6150 5200 50  0000 C CNN
-F 2 "" H 6150 5350 50  0000 C CNN
-F 3 "" H 6150 5350 50  0000 C CNN
-	1    6150 5350
-	1    0    0    -1
-$EndComp
-Text GLabel 6750 5350 2    60   Input ~ 0
+P 6700 5350
+F 0 "#PWR033" H 6700 5100 50  0001 C CNN
+F 1 "GND" H 6700 5200 50  0000 C CNN
+F 2 "" H 6700 5350 50  0000 C CNN
+F 3 "" H 6700 5350 50  0000 C CNN
+	1    6700 5350
+	1    0    0    -1
+$EndComp
+Text GLabel 7300 5350 2    60   Input ~ 0
 AUX_BUTTON
 Text GLabel 2250 2250 2    60   Input ~ 0
@@
 F 0 "U8" H 9950 5460 50  0000 L BNN
 F 1 "DS18B20" H 9950 4840 50  0000 L BNN
-F 2 "TO-92-AMMO" H 10250 5150 50  0001 L BNN
+F 2 "homebrew:TO-92" H 10250 5150 50  0001 L BNN
 F 3 "DS18B20+T&amp;R" H 10250 5150 50  0001 L BNN
 F 4 "TO-226-3 Maxim Integrated" H 10250 5150 50  0001 L BNN "Field4"
@@
 INTERNAL_TEMP
 $Comp
-L VCC #PWR036
+L VCC #PWR034
 U 1 1 5B531E6E
 P 9850 4950
-F 0 "#PWR036" H 9850 4800 50  0001 C CNN
+F 0 "#PWR034" H 9850 4800 50  0001 C CNN
 F 1 "VCC" H 9850 5100 50  0000 C CNN
 F 2 "" H 9850 4950 50  0000 C CNN
@@
 $EndComp
 $Comp
-L GND #PWR037
+L GND #PWR035
 U 1 1 5B531ED0
 P 9850 5350
-F 0 "#PWR037" H 9850 5100 50  0001 C CNN
+F 0 "#PWR035" H 9850 5100 50  0001 C CNN
 F 1 "GND" H 9850 5200 50  0000 C CNN
 F 2 "" H 9850 5350 50  0000 C CNN
@@
 $EndComp
 $Comp
-L VCC #PWR038
+L VCC #PWR036
 U 1 1 5B531FCE
 P 9850 5700
-F 0 "#PWR038" H 9850 5550 50  0001 C CNN
+F 0 "#PWR036" H 9850 5550 50  0001 C CNN
 F 1 "VCC" H 9850 5850 50  0000 C CNN
 F 2 "" H 9850 5700 50  0000 C CNN
@@
 $EndComp
 $Comp
-L GND #PWR039
+L GND #PWR037
 U 1 1 5B532030
 P 9300 5900
-F 0 "#PWR039" H 9300 5650 50  0001 C CNN
+F 0 "#PWR037" H 9300 5650 50  0001 C CNN
 F 1 "GND" H 9300 5750 50  0000 C CNN
 F 2 "" H 9300 5900 50  0000 C CNN
@@
 F 0 "P2" H 10050 6500 50  0000 C CNN
 F 1 "CONN_01X08" V 10150 6050 50  0000 C CNN
-F 2 "" H 10050 6050 50  0000 C CNN
+F 2 "homebrew:1985250_phoenix_8pos_3.5mm" H 10050 6050 50  0001 C CNN
 F 3 "" H 10050 6050 50  0000 C CNN
 	1    10050 6050
@@
 FLOAT_SWITCH
 $Comp
-L GND #PWR040
+L GND #PWR038
 U 1 1 5B533A48
 P 9850 6400
-F 0 "#PWR040" H 9850 6150 50  0001 C CNN
+F 0 "#PWR038" H 9850 6150 50  0001 C CNN
 F 1 "GND" H 9850 6250 50  0000 C CNN
 F 2 "" H 9850 6400 50  0000 C CNN
@@
 NoConn ~ 9850 6200
 NoConn ~ 2250 1250
+$Comp
+L POT-RESCUE-hvac-v2 RV2
+U 1 1 5B536446
+P 4050 5150
+F 0 "RV2" V 3875 5150 50  0000 C CNN
+F 1 "POT" V 3950 5150 50  0000 C CNN
+F 2 "homebrew:BOURNS_PDB12H_POT" H 4050 5150 50  0001 C CNN
+F 3 "" H 4050 5150 50  0001 C CNN
+	1    4050 5150
+	1    0    0    -1
+$EndComp
+$Comp
+L VCC #PWR039
+U 1 1 5B53644C
+P 4050 5000
+F 0 "#PWR039" H 4050 4850 50  0001 C CNN
+F 1 "VCC" H 4050 5150 50  0000 C CNN
+F 2 "" H 4050 5000 50  0001 C CNN
+F 3 "" H 4050 5000 50  0001 C CNN
+	1    4050 5000
+	1    0    0    -1
+$EndComp
+$Comp
+L GND #PWR040
+U 1 1 5B536452
+P 4050 5300
+F 0 "#PWR040" H 4050 5050 50  0001 C CNN
+F 1 "GND" H 4050 5150 50  0000 C CNN
+F 2 "" H 4050 5300 50  0001 C CNN
+F 3 "" H 4050 5300 50  0001 C CNN
+	1    4050 5300
+	1    0    0    -1
+$EndComp
 $EndSCHEMATC

Commit message: Associate footprints
Parts:
- SW3, SW4: value SW_PUSH -> KS-01Q-01; footprint (none) -> homebrew:BUTTON_KS-01Q-01
- SW5: footprint (none) -> homebrew:SWITCH_100SP1T2B3M1QEH
Changed lines of the file:
@@
 P 7000 5050
 F 0 "SW3" H 7150 5160 50  0000 C CNN
-F 1 "SW_PUSH" H 7000 4970 50  0000 C CNN
-F 2 "" H 7000 5050 50  0001 C CNN
+F 1 "KS-01Q-01" H 7000 4970 50  0000 C CNN
+F 2 "homebrew:BUTTON_KS-01Q-01" H 7000 5050 50  0001 C CNN
 F 3 "" H 7000 5050 50  0000 C CNN
 	1    7000 5050
@@
 F 0 "SW5" H 9000 950 50  0000 C CNN
 F 1 "SPST" H 9000 750 50  0000 C CNN
-F 2 "" H 9000 850 50  0001 C CNN
+F 2 "homebrew:SWITCH_100SP1T2B3M1QEH" H 9000 850 50  0001 C CNN
 F 3 "" H 9000 850 50  0000 C CNN
 	1    9000 850
@@
 P 7000 5350
 F 0 "SW4" H 7150 5460 50  0000 C CNN
-F 1 "SW_PUSH" H 7000 5270 50  0000 C CNN
-F 2 "" H 7000 5350 50  0001 C CNN
+F 1 "KS-01Q-01" H 7000 5270 50  0000 C CNN
+F 2 "homebrew:BUTTON_KS-01Q-01" H 7000 5350 50  0001 C CNN
 F 3 "" H 7000 5350 50  0000 C CNN
 	1    7000 5350

Commit message: Route power (GIANT TRACES)
Connections:
- net KNOB renamed SPEED
Changed lines of the file:
@@
 MODE
 Text GLabel 2250 1550 2    60   Input ~ 0
-KNOB
+SPEED
 $Comp
 L POT-RESCUE-hvac-v2 RV1
@@
 $EndComp
 Text GLabel 5500 5150 2    60   Input ~ 0
-KNOB
+SPEED
 NoConn ~ 2250 1050
 NoConn ~ 2250 1150

Commit message: Place the programming header and diode
Parts:
- D1: footprint Diodes_SMD:D_SOD-123 -> Diodes_SMD:SOD-123
- J1: footprint Pin_Headers:Pin_Header_Straight_1x04_Pitch2.54mm -> Pin_Headers:Pin_Header_Straight_1x04
Changed lines of the file:
@@
 F 0 "J1" H 2750 7250 50  0000 C CNN
 F 1 "Conn_01x04" H 2750 6750 50  0000 C CNN
-F 2 "Pin_Headers:Pin_Header_Straight_1x04_Pitch2.54mm" H 2750 7050 50  0001 C CNN
+F 2 "Pin_Headers:Pin_Header_Straight_1x04" H 2750 7050 50  0001 C CNN
 F 3 "" H 2750 7050 50  0001 C CNN
 	1    2750 7050
@@
 F 0 "D1" H 1100 6850 50  0000 C CNN
 F 1 "BAT54GWJ" H 1100 6650 50  0000 C CNN
-F 2 "Diodes_SMD:D_SOD-123" H 1100 6750 50  0001 C CNN
+F 2 "Diodes_SMD:SOD-123" H 1100 6750 50  0001 C CNN
 F 3 "" H 1100 6750 50  0001 C CNN
 	1    1100 6750

Commit message: Hardware revision 2.1: - Fix SWD connection to power to not connect directly to VCC - Add silk labels for controls
Connections:
- net VCC: no longer J1.1 (Pin_1)
- net USB_VCC: now reaches D1.2 (A), P1.1 (VCC)
- net USB_VCC: now also J1.1 (Pin_1)
Other:
- moved on the sheet: D1
Changed lines of the file:
@@
 LIBS:switches
 LIBS:relays
+LIBS:motors
 LIBS:transistors
 LIBS:conn
@@
 LIBS:contrib
 LIBS:valves
-LIBS:homebrew
 LIBS:hvac-v2-cache
 EELAYER 25 0
@@
 L +BATT #PWR06
 U 1 1 5B4EC5AA
-P 1100 6600
-F 0 "#PWR06" H 1100 6450 50  0001 C CNN
-F 1 "+BATT" H 1100 6740 50  0000 C CNN
-F 2 "" H 1100 6600 50  0001 C CNN
-F 3 "" H 1100 6600 50  0001 C CNN
-	1    1100 6600
+P 850 6600
+F 0 "#PWR06" H 850 6450 50  0001 C CNN
+F 1 "+BATT" H 850 6740 50  0000 C CNN
+F 2 "" H 850 6600 50  0001 C CNN
+F 3 "" H 850 6600 50  0001 C CNN
+	1    850  6600
 	1    0    0    -1
 $EndComp
@@
 F 3 "" H 5250 7150 50  0001 C CNN
 	1    5250 7150
-	1    0    0    -1
-$EndComp
-$Comp
-L VCC #PWR012
-U 1 1 5B4ED9BB
-P 2550 6950
-F 0 "#PWR012" H 2550 6800 50  0001 C CNN
-F 1 "VCC" H 2550 7100 50  0000 C CNN
-F 2 "" H 2550 6950 50  0001 C CNN
-F 3 "" H 2550 6950 50  0001 C CNN
-	1    2550 6950
 	1    0    0    -1
 $EndComp
@@
 L D D1
 U 1 1 5B516D29
-P 1100 6750
-F 0 "D1" H 1100 6850 50  0000 C CNN
-F 1 "BAT54GWJ" H 1100 6650 50  0000 C CNN
-F 2 "Diodes_SMD:SOD-123" H 1100 6750 50  0001 C CNN
-F 3 "" H 1100 6750 50  0001 C CNN
-	1    1100 6750
+P 850 6750
+F 0 "D1" H 850 6850 50  0000 C CNN
+F 1 "BAT54GWJ" H 850 6650 50  0000 C CNN
+F 2 "Diodes_SMD:SOD-123" H 850 6750 50  0001 C CNN
+F 3 "" H 850 6750 50  0001 C CNN
+	1    850  6750
 	0    1    1    0
 $EndComp
@@
 	6050 2750 6000 2750
 Wire Wire Line
-	1150 6950 1100 6950
+	850  6950 1150 6950
 Wire Wire Line
 	1100 6950 1100 6900
@@
 	1    0    0    -1
 $EndComp
+Wire Wire Line
+	850  6950 850  6900
+Connection ~ 1100 6950
+Text GLabel 1100 6900 1    60   Input ~ 0
+USB_VCC
+Text GLabel 2550 6950 0    60   Input ~ 0
+USB_VCC
 $EndSCHEMATC
