File: hvac-v2.sch (KiCad schematic (older format))
At the start: 24 parts, among them J2 Anderson_two_redblack, J3 Anderson_two_redblack, J4 Anderson_two_redblack, SW5 SPST

Commit message: Start adding motor drivers
Parts:
- added C? (x4): 0.1uF, Capacitor_SMD:C_0402_1005Metric, symbol Device:C
- added D? (x2): D_Schottky, Diode_THT:D_DO-201AD_P12.70mm_Horizontal, symbol Device:D_Schottky
- added D? (x2): D_TVS, Diode_SMD:D_SOD-323, symbol Device:D_TVS
- added JP? (x2): SolderJumper_2_Open, symbol Jumper:SolderJumper_2_Open
- added Q? (x2): AO3400A, Package_TO_SOT_SMD:SOT-23, symbol Transistor_FET:AO3400A
- added R? (x2): 150, Resistor_SMD:R_0603_1608Metric, symbol Device:R
- added R? (x2): 24k, Resistor_SMD:R_0603_1608Metric, symbol Device:R
- added R? (x2): 10k, Resistor_SMD:R_0603_1608Metric, symbol Device:R
- added U? (x2): IFX007T, symbol Homebrew:IFX007T
Connections:
- net +BATT: now also C?.1, C?.1, D?.1 (K), D?.1 (K), JP?.2 (B); no longer J3.1
- net GND: now also C?.2, C?.2, D?.2 (A2), D?.2 (A2), Q?.2 (S), Q?.2 (S)
- net PUMP_OUT: now also C?.2, D?.2 (A), Q?.3 (D), R?.1
- net PUMP_SENSE: now reaches U?.11 (PA1)
- net PUMP_SENSE: now also C?.1, C?.1, D?.1 (A1), D?.1 (A1), R?.2, R?.2
- net FAN_SIGNAL: now reaches U?.16 (PA6)
- net FAN_SIGNAL: now also R?.2
- net PUMP_SIGNAL: now reaches U?.17 (PA7)
- net PUMP_SIGNAL: now also R?.2
- net FAN_OUT renamed FAN_L
- new net: Q?.1 (G), R?.1 (x2)
- new net: R?.2, U?.2 (IN)
- new net: R?.2, U?.3 (INH)
- new net: U?.4 (OUT), U?.8 (OUT) (x2)
- new net: C?.2, D?.2 (A), JP?.1 (A), Q?.3 (D), R?.1
- new net FAN_N: JP?.2 (B)
- new net FAN_P: J3.1, JP?.1 (A)
Other:
- moved on the sheet: H1, H2, H3, H4, J4

Commit message: Finish updating schematic for JLC assembly
Parts:
- removed J2, J4: Anderson_two_redblack, homebrew:Anderson_1337G3_right_angle_bottom_two, symbol hvac-v2-rescue:Anderson_two_redblack
- removed SW5: SPST, homebrew:SWITCH_100SP1T2B3M1QEH, symbol hvac-v2-rescue:SPST
- added BZ1: Buzzer, homebrew:MURATA_PKM13EPYH4000-A0, symbol Device:Buzzer
- added C10, C11, C15, C16: 0.22uF, Capacitor_SMD:C_0805_2012Metric, symbol Device:C
- added C12, C13, C18, C21, C22, C23, C24, C26, C27, C28, C29, C30, C31, C32, C34, C35, C36, C37, C40, C41, C42, C43, C7: 0.1uF, Capacitor_SMD:C_0402_1005Metric, symbol Device:C
- added C19, C39: 1000uF, Capacitor_THT:CP_Radial_D10.0mm_P5.00mm, symbol Device:CP
- added C20, C3: 1nF, Capacitor_SMD:C_0402_1005Metric, symbol Device:C
- added C38: 4.7uF, Capacitor_SMD:C_0603_1608Metric, symbol Device:C
- added D10, D12, D13, D14, D15, D19, D20, D21, D22, D23, D24, D6, D7: TVS_5V, Diode_SMD:D_SOD-323, symbol Device:D_TVS
- added D16, D18, D8, D9: D_Schottky, Diode_THT:D_DO-201AD_P12.70mm_Horizontal, symbol Device:D_Schottky
- added D5: LED, LED_SMD:LED_0805_2012Metric, symbol Device:LED
- added J10, J3, J9: Conn_01x02, Connector_PinHeader_2.54mm:PinHeader_1x02_P2.54mm_Horizontal, symbol Connector_Generic:Conn_01x02
- added J11, J12, J13, J5, J6: Conn_01x03, Connector_PinHeader_2.54mm:PinHeader_1x03_P2.54mm_Horizontal, symbol Connector_Generic:Conn_01x03
- added J14: Conn_01x04, Connector_PinHeader_2.54mm:PinHeader_1x04_P2.54mm_Horizontal, symbol Connector_Generic:Conn_01x04
- added J4: Anderson_two_redblack_src, homebrew:Anderson_1336G1_right_angle_bottom_two, symbol Homebrew:Anderson_two_redblack_src
- added J7, J8: Anderson_two_redblack_sink, homebrew:Anderson_1336G1_right_angle_bottom_two, symbol Homebrew:Anderson_two_redblack_sink
- added Q3: AO3400A, Package_TO_SOT_SMD:SOT-23, symbol Transistor_FET:AO3400A
- added R1, R14: 470, Resistor_SMD:R_0603_1608Metric, symbol Device:R
- added R10, R11, R12, R17, R18, R19, R20, R5: 10k, Resistor_SMD:R_0603_1608Metric, symbol Device:R
- added R13, R15, R24: 150, Resistor_SMD:R_0603_1608Metric, symbol Device:R
- added R16: 47, Resistor_SMD:R_0603_1608Metric, symbol Device:R
- added R22: 24k, Resistor_SMD:R_0603_1608Metric, symbol Device:R
- added R25, R26, R27, R28: 4k7, Resistor_SMD:R_0603_1608Metric, symbol Device:R
- added SW2: Rotary_Encoder_Switch, homebrew:BOURNS_PEC12R-4xxxF-Sxxxx, symbol Device:Rotary_Encoder_Switch
- added U4: AMS1117-3.3, Package_TO_SOT_SMD:SOT-223-3_TabPin2, symbol Regulator_Linear:AMS1117-3.3
- added U5: DS18B20, Package_TO_SOT_THT:TO-92_Inline, symbol Sensor_Temperature:DS18B20
- D1, D11, D2: renamed from D?; value D_TVS -> TVS_5V; LCSC (none) -> C182013; MPN DESD5V0U1BA-7 -> (none)
- D4: renamed from D?; value D_TVS -> TVS_12V; footprint Diode_SMD:D_SOD-323 -> Diode_SMD:D_SMB_Handsoldering; MPN DESD5V0U1BA-7 -> SMBJ16CA
- F1: footprint homebrew:FUSEHOLDER_ATC_Bk-6010 -> homebrew:FUSE_3550-2; MPN (none) -> 3550-2
- J2: renamed from J?; footprint (none) -> Connector_PinHeader_2.54mm:PinHeader_1x04_P2.54mm_Horizontal
- JP1, JP2: renamed from JP?; footprint (none) -> Jumper:SolderJumper-2_P1.3mm_Open_TrianglePad1.0x1.5mm
- SW1: renamed from SW?; footprint (none) -> homebrew:SW_TACTILE_5.1MM_TS-1187A-C-D-B; LCSC (none) -> C318884
- U1: renamed from U?; LCSC (none) -> C23922
- U2, U3: renamed from U?; footprint (none) -> Package_TO_SOT_SMD:TO-263-7_TabPin8; MPN (none) -> IFX007T
- gave numbers to parts that had none: 24
- renumbered J3 to J1
Connections:
- net FAN_L is gone; now on net FAN_N: J1.2
- net +BATT: now also D4.1 (A1), F1.2 (OUT), R8.1, U2.7 (VS), U3.7 (VS), C10.1, C12.1, C13.2, C15.2, C19.1, C30.2, C34.1, D16.1 (K), D18.1 (K), J7.1, J8.1, U4.3 (VI); no longer C17.1, D3.1 (K), R9.1
- net BOOT0: now also U1.44 (BOOT0)
- net FAN_N: now also C17.2, D3.2 (A), U3.4 (OUT), U3.8 (OUT), C15.1, C16.2
- net FAN_P: now also C17.1, D3.1 (K), U2.4 (OUT), U2.8 (OUT), C10.2, C11.1
- net FAN_SIGNAL: now also U1.30 (PA9); no longer U1.16 (PA6)
- net GND: now also R9.2, U2.1 (GND), U3.1 (GND), BZ1.2 (+), C11.2, C12.2, C13.1, C16.1, C18.2, C19.2, C20.2, C21.2, C22.2, C23.2, C24.2, C26.2, C27.1, C28.2, C29.2, C3.2, C30.1, C31.2, C32.2, C35.2, C36.2, C37.2, C38.2, C39.2, C40.2, C41.2, C42.2, C43.2, C7.1, D10.2 (A2), D12.2 (A2), D13.2 (A2), D14.2 (A2), D15.2 (A2), D19.2 (A2), D20.2 (A2), D21.2 (A2), D22.2 (A2), D23.2 (A2), D24.2 (A2), D6.1 (A1), D7.1 (A1), D8.2 (A), D9.2 (A), J10.1 (Pin_1), J11.1 (Pin_1), J12.1 (Pin_1), J13.1 (Pin_1), J14.3 (Pin_3), J3.2 (Pin_2), J4.2, J5.1 (Pin_1), J6.1 (Pin_1), J9.1 (Pin_1), Q3.2 (S), R1.2, R10.2, R13.1, R14.2, R5.2, SW2.C, SW2.S2, U4.1 (GND), U5.1 (GND); no longer R8.2
- net PUMP_OUT: now also J7.2
- net PUMP_SENSE: now also U1.15 (PA5); no longer C6.1, D1.1 (A1), R6.2
- net PUMP_SIGNAL: now also U1.31 (PA10); no longer U1.17 (PA7)
- net VBATT_DIV: now also R8.2, R9.1, U1.14 (PA4); no longer R8.1, R9.2
- net VCC: now also C35.1, C36.1, C37.1, C38.1, C39.1, C40.1, C41.1, C42.1, C43.1, D16.2 (A), D21.1 (A1), J11.3 (Pin_3), J12.3 (Pin_3), J13.3 (Pin_3), J14.4 (Pin_4), J5.3 (Pin_3), J6.3 (Pin_3), R18.1, R19.2, R25.1, R26.1, R27.1, R28.1, U4.2 (VO), U5.3 (VDD)
- net at F1.1 (IN): now also D8.1 (K), D9.1 (K), J4.1
- net BRIDGE_SENSE_P: now reaches U1.12 (PA2)
- net BRIDGE_SENSE_P: now also U2.6 (IS), C3.1, R1.1
- net BRIDGE_SENSE_N: now reaches U1.13 (PA3)
- net BRIDGE_SENSE_N: now also U3.6 (IS), C20.1, R14.1
- net BRIDGE_ENABLE: now reaches U1.18 (PB0)
- net BRIDGE_ENABLE: now also R4.1, R11.2
- net BUZZER: now reaches U1.19 (PB1)
- net BUZZER: now also R16.1
- net BRIDGE_N: now reaches U1.20 (PB2)
- net BRIDGE_N: now also R12.2
- net ENC_A: now reaches U1.27 (PB14)
- net ENC_A: now also C21.1, D7.2 (A2), R17.2
- net ENC_B: now reaches U1.28 (PB15)
- net ENC_B: now also C27.2, D13.1 (A1), R20.1
- net PWM_OUT: now reaches U1.29 (PA8)
- net PWM_OUT: now also R15.1
- net LED: now reaches U1.32 (PA11)
- net LED: now also D5.2 (A)
- net SWDIO: now reaches U1.34 (PA13)
- net SWDIO: now also J14.2 (Pin_2)
- net SWCLK: now reaches U1.37 (PA14)
- net SWCLK: now also J14.1 (Pin_1)
- net BRIDGE_P: now reaches U1.39 (PB3)
- net BRIDGE_P: now also R3.1
- net TEMP_BUILTIN: now reaches U1.41 (PB5)
- net TEMP_BUILTIN: now also R25.2, U5.2 (DQ)
- net TEMP_INSIDE: now reaches U1.42 (PB6)
- net TEMP_INSIDE: now also D22.1 (A1), J11.2 (Pin_2), R26.2
- net TEMP_OUTSIDE: now reaches U1.43 (PB7)
- net TEMP_OUTSIDE: now also D23.1 (A1), J12.2 (Pin_2), R27.2
- net TEMP_AUX: now reaches U1.45 (PB8)
- net TEMP_AUX: now also D24.1 (A1), J13.2 (Pin_2), R28.2
- net ACC_SIGNAL: now reaches U1.46 (PB9)
- net ACC_SIGNAL: now also R24.2
- net at U2.5 (SR): now also C7.2, R5.1
- net at U3.2 (IN): now also R12.1
- net at U3.3 (INH): now also R11.1
- net at U3.5 (SR): now also C18.1, R10.1
- net at JP2.1 (A), Q1.3 (D), R6.1: no longer C17.2, D3.2 (A)
- new net: D5.1 (K), R13.2
- new net: D6.2 (A2), J3.1 (Pin_1), R15.2
- new net: Q3.1 (G), R24.1
- new net: R19.1, R20.2, SW2.A
- new net: R17.1, R18.2, SW2.B
- new net: BZ1.1 (-), C22.1, C23.1, R16.2
- new net ACC_OUT: C34.2, D18.2 (A), J8.2, Q3.3 (D), R22.1
- new net ACC_SENSE: C26.1, D12.1 (A1), R22.2, U1.17 (PA7)
- new net BUTTON: C24.1, D10.1 (A1), SW2.S1
- new net FAN_SENSE: C6.1, D1.1 (A1), R6.2, U1.16 (PA6)
- new net SW_1: C32.1, D20.1 (A1), J10.2 (Pin_2)
- new net SW_2: C28.1, D14.1 (A1), J5.2 (Pin_2)
- new net SW_3: C29.1, D15.1 (A1), J6.2 (Pin_2)
- new net SW_WATER: C31.1, D19.1 (A1), J9.2 (Pin_2)
- no-connect marks 0 -> 12
Other:
- note added: "Fc=17kHz"
- moved on the sheet: C14, C17, C25, C33, C6, D1, D11, D17, D2, D3, D4, H1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

Commit message: Start placing components
Parts:
- J1: footprint homebrew:Anderson_1337G3_right_angle_bottom_two -> homebrew:Anderson_1336G1_right_angle_bottom_two
Changed lines of the file:
@@
 F 0 "J1" H 6850 9750 60  0000 C CNN
 F 1 "Anderson_two_redblack" H 6850 10050 60  0000 C CNN
-F 2 "homebrew:Anderson_1337G3_right_angle_bottom_two" H 6800 9750 60  0001 C CNN
+F 2 "homebrew:Anderson_1336G1_right_angle_bottom_two" H 6800 9750 60  0001 C CNN
 F 3 "" H 6800 9750 60  0001 C CNN
 	1    6850 9900

Commit message: Component placement finished
Parts:
- added H5: HOLE, homebrew:HOLE_M4, symbol hvac-v2-rescue:HOLE
- added R29, R31: 110k, Resistor_SMD:R_0603_1608Metric, symbol Device:R
- added R30, R32, R33: 10k, Resistor_SMD:R_0603_1608Metric, symbol Device:R
- added R34, R35, R36, R37: 150, Resistor_SMD:R_0603_1608Metric, symbol Device:R
- C19, C39: MPN 860010475017 -> 25PK1000MEFC10X16
- F1: value BK-6010 -> ATC
Connections:
- net ACC_SIGNAL: now also R33.1
- net BRIDGE_ENABLE: now also R29.1, R31.1
- net FAN_SIGNAL: now also R30.1
- net GND: now also R29.2, R30.2, R31.2, R32.2, R33.2
- net PUMP_SIGNAL: now also R32.1
- net SW_1: now also U1.22 (PB11), R36.2; no longer C32.1, D20.1 (A1), J10.2 (Pin_2)
- net SW_2: now also U1.25 (PB12), R34.2; no longer C28.1, D14.1 (A1), J5.2 (Pin_2)
- net SW_3: now also U1.26 (PB13), R35.2; no longer C29.1, D15.1 (A1), J6.2 (Pin_2)
- net SW_WATER: now also U1.21 (PB10), R37.2; no longer C31.1, D19.1 (A1), J9.2 (Pin_2)
- new net: C31.1, D19.1 (A1), J9.2 (Pin_2), R37.1
- new net: C32.1, D20.1 (A1), J10.2 (Pin_2), R36.1
- new net: C28.1, D14.1 (A1), J5.2 (Pin_2), R34.1
- new net: C29.1, D15.1 (A1), J6.2 (Pin_2), R35.1
- no-connect marks 12 -> 8
Other:
- moved on the sheet: C31, C32, C36, C37, D19, D20, J10, J9, R12, R3

Commit message: Start routing
Parts:
- added H6: SLOT, homebrew:SLOT_W2mm_H8mm, symbol hvac-v2-rescue:HOLE
Changed lines of the file:
@@
 Text Label 1700 4250 2    50   ~ 0
 SW_3
+$Comp
+L hvac-v2-rescue:HOLE H6
+U 1 1 6265A8C4
+P 14750 800
+F 0 "H6" H 14750 670 60  0000 C CNN
+F 1 "SLOT" H 14750 920 60  0000 C CNN
+F 2 "homebrew:SLOT_W2mm_H8mm" H 14750 800 60  0001 C CNN
+F 3 "" H 14750 800 60  0001 C CNN
+	1    14750 800
+	1    0    0    -1
+$EndComp
 $EndSCHEMATC
