File: hvac-v2.kicad_sch (KiCad schematic)
At the start: 138 parts

Commit message: First pass at routing
Parts:
- removed R31: (no value), symbol Device:R
- added C44, C45: 0.1uF, Capacitor_SMD:C_0402_1005Metric, symbol Device:C
- added C46: 4.7uF, Capacitor_SMD:C_0603_1608Metric, symbol Device:C
- added D25: D_Schottky, Diode_THT:D_DO-201AD_P12.70mm_Horizontal, symbol Device:D_Schottky
- added D26: TVS_5V, Diode_SMD:D_SOD-323, symbol Device:D_TVS
- added U6: (no value), symbol Regulator_Linear:AMS1117-5.0
- C19, C39: symbol Device:CP -> Device:C_Polarized
- SW2: symbol Device:Rotary_Encoder_Switch -> Device:RotaryEncoder_Switch
Connections:
- net +BATT: now also C44.2, D25.1 (K), U6.3 (VI)
- net GND: now also C44.1, C45.2, C46.2, D26.2 (A2), U6.1 (GND)
- net PUMP_SENSE: no longer U1.15 (PA5)
- net SW_2: now also U1.26 (PB13); no longer U1.25 (PB12)
- net SW_3: now also U1.25 (PB12); no longer U1.26 (PB13)
- net VBATT_DIV: no longer U1.14 (PA4)
- net VCC: no longer C37.1, J2.3 (Pin_3), J6.3 (Pin_3)
- new net +5V: C37.1, C45.1, C46.1, D25.2 (A), D26.1 (A1), J2.3 (Pin_3), J6.3 (Pin_3), U6.2 (VO)
- no-connect marks 8 -> 10
Other:
- moved on the sheet: C30, C35, C38, C39, D16, D21, U4
